Commit message: Changes to model. Added PID control

File: src/autonomous_drone/description/material.xacro (robot description, xacro)
@@ -18,4 +18,7 @@
 	<material name="golden">
 		<color rgba="${212/255} ${175/255} ${55/255} 1" />
+	</material>
+	<material name="yellow">
+		<color rgba="0.8 0.8 0.01 1" />
 	</material>
 	<!-- ================================= -->
@@ -57,3 +60,18 @@
 		<material>Gazebo/Black</material>
 	</gazebo>
+	<gazebo reference="arduino" >
+		<material>Gazebo/Blue</material>
+	</gazebo>
+	<gazebo reference="ESC1" >
+		<material>Gazebo/Yellow</material>
+	</gazebo>
+	<gazebo reference="ESC2" >
+		<material>Gazebo/Yellow</material>
+	</gazebo>
+	<gazebo reference="ESC3" >
+		<material>Gazebo/Yellow</material>
+	</gazebo>
+	<gazebo reference="ESC4" >
+		<material>Gazebo/Yellow</material>
+	</gazebo>
 </robot>

File: src/autonomous_drone/description/quadcopter.urdf.xacro (robot description, xacro)
@@ -25,8 +25,12 @@
 	</xacro:macro>
 <!-- ======================================================== -->
-    <!-- BASE_FOOTPRINT LINK -->
+    <!-- BASE LINK -->
     <link name="base_link">
     </link>
 <!-- ======================================================== -->
+    <!-- BASE_FOOTPRINT LINK -->
+	<link name="base_footprint">
+    </link>
+<!-- ======================================================== -->
 	<link name="base_link1">
 		<visual>
@@ -163,4 +167,88 @@
 		</collision>
 		<xacro:default_inertial mass="${0.01}" p="${0}" ix_value="${8.95e-6}" iy_value="${8.95e-6}" iz_value="${2.23e-4}" />
+	</link>
+<!-- ======================================================== -->
+<link name="arduino">
+		<visual>
+			<origin xyz="0 0 0" rpy="0 0 0" />
+			<geometry>
+				<box size="0.1 0.1 0.001" />
+			</geometry>
+		</visual>
+		<collision>
+			<origin xyz="0 0 0" rpy="0 0 0" />
+			<geometry>
+				<box size="0.1 0.1 0.001" />
+			</geometry>
+		</collision>
+		<xacro:default_inertial mass="${0.01}" p="${0}" ix_value="${0}" iy_value="${0}" iz_value="${8.33333e-5}" />
+	</link>
+<!-- ======================================================== -->
+	<link name="ESC1">
+		<visual>
+			<origin xyz="0 0 0" rpy="0 0 ${-pi_value/4}" />
+			<geometry>
+				<box size="${width} ${0.07} ${0.008}" />
+			</geometry>
+			<material name="yellow" />
+		</visual>
+		<collision>
+			<origin xyz="0 0 0" rpy="0 0 ${-pi_value/4}" />
+			<geometry>
+				<box size="${width} ${0.07} ${0.008}" />
+			</geometry>
+		</collision>
+		<xacro:default_inertial mass="${0.01}" p="${-pi_value/4}" ix_value="${0}" iy_value="${0}" iz_value="${3.664e-5}" />
+	</link>
+<!-- ======================================================== -->
+	<link name="ESC2">
+		<visual>
+			<origin xyz="0 0 0" rpy="0 0 ${-pi_value/4}" />
+			<geometry>
+				<box size="${width} ${0.07} ${0.008}" />
+			</geometry>
+			<material name="yellow" />
+		</visual>
+		<collision>
+			<origin xyz="0 0 0" rpy="0 0 ${-pi_value/4}" />
+			<geometry>
+				<box size="${width} ${0.07} ${0.008}" />
+			</geometry>
+		</collision>
+		<xacro:default_inertial mass="${0.01}" p="${-pi_value/4}" ix_value="${0}" iy_value="${0}" iz_value="${3.664e-5}" />
+	</link>
+<!-- ======================================================== -->
+	<link name="ESC3">
+		<visual>
+			<origin xyz="0 0 0" rpy="0 0 ${pi_value/4}" />
+			<geometry>
+				<box size="${width} ${0.07} ${0.008}" />
+			</geometry>
+			<material name="yellow" />
+		</visual>
+		<collision>
+			<origin xyz="0 0 0" rpy="0 0 ${pi_value/4}" />
+			<geometry>
+				<box size="${width} ${0.07} ${0.008}" />
+			</geometry>
+		</collision>
+		<xacro:default_inertial mass="${0.01}" p="${pi_value/4}" ix_value="${0}" iy_value="${0}" iz_value="${3.664e-5}" />
+	</link>
+<!-- ======================================================== -->
+	<link name="ESC4">
+		<visual>
+			<origin xyz="0 0 0" rpy="0 0 ${pi_value/4}" />
+			<geometry>
+				<box size="${width} ${0.07} ${0.008}" />
+			</geometry>
+			<material name="yellow" />
+		</visual>
+		<collision>
+			<origin xyz="0 0 0" rpy="0 0 ${pi_value/4}" />
+			<geometry>
+				<box size="${width} ${0.07} ${0.008}" />
+			</geometry>
+		</collision>
+		<xacro:default_inertial mass="${0.01}" p="${pi_value/4}" ix_value="${0}" iy_value="${0}" iz_value="${3.664e-5}" />
 	</link>
 <!-- ======================================================== -->
@@ -230,4 +318,11 @@
 		<xacro:default_inertial mass="${mass_pr}" p="${0}"  ix_value="${0}" iy_value="${0}" iz_value="${4.42448e-5}" />
 	</link>
+<!-- ======================================================== -->
+    <!-- Define the joint between the base and footprint -->
+	<joint name="base_footprint_joint" type="fixed">
+        <parent link="base_link"/>
+        <child link="base_footprint"/>
+        <origin xyz="0 0 0" rpy="0 0 0"/>
+    </joint>
 <!-- ======================================================== -->
 	<!-- Define the joint between the arms of the frame -->
@@ -322,4 +417,44 @@
 		<child link="cyl4" />
 		<origin xyz="${prop_loc - 0.01} ${-prop_loc + 0.01} 0.01" rpy="0 0 0" />
+		<axis xyz="0 0 1" />
+	</joint>
+<!-- ======================================================== -->
+<!-- Define joint between Arduino and frame -->
+	<joint name="joint_arduino_frame" type="fixed">
+		<parent link="plate2" />
+		<child link="arduino" />
+		<origin xyz="${0} ${0} 0.005" rpy="0 0 0" />
+		<axis xyz="0 0 1" />
+	</joint>
+<!-- ======================================================== -->
+<!-- Define joint between ESC and frame -->
+	<joint name="joint_frame_ESC1" type="fixed">
+		<parent link="base_link2" />
+		<child link="ESC1" />
+		<origin xyz="${prop_loc/2 + 0.013} ${prop_loc/2 + 0.013} 0.009" rpy="0 0 0" />
+		<axis xyz="0 0 1" />
+	</joint>
+<!-- ======================================================== -->
+<!-- Define joint between ESC and frame -->
+	<joint name="joint_frame_ESC2" type="fixed">
+		<parent link="base_link2" />
+		<child link="ESC2" />
+		<origin xyz="${-prop_loc/2 - 0.013} ${-prop_loc/2 - 0.013} 0.009" rpy="0 0 0" />
+		<axis xyz="0 0 1" />
+	</joint>
+<!-- ======================================================== -->
+<!-- Define joint between ESC and frame -->
+	<joint name="joint_frame_ESC3" type="fixed">
+		<parent link="base_link1" />
+		<child link="ESC3" />
+		<origin xyz="${-prop_loc/2 - 0.013} ${prop_loc/2 + 0.013} 0.009" rpy="0 0 0" />
+		<axis xyz="0 0 1" />
+	</joint>
+<!-- ======================================================== -->
+<!-- Define joint between ESC and frame -->
+	<joint name="joint_frame_ESC4" type="fixed">
+		<parent link="base_link1" />
+		<child link="ESC4" />
+		<origin xyz="${prop_loc/2 + 0.013} ${-prop_loc/2 - 0.013} 0.009" rpy="0 0 0" />
 		<axis xyz="0 0 1" />
 	</joint>
