Commit message: Added Slam Support but PID still not working

File: src/autonomous_drone/description/lidar.xacro (robot description, xacro)
@@ -58,4 +58,7 @@
             </ray>
             <plugin name="laser_controller" filename="libgazebo_ros_ray_sensor.so">
+                <ros>
+                    <argument>~/out:=scan</argument>
+                </ros>
                 <output_type>sensor_msgs/LaserScan</output_type>
                 <frame_name>laser_frame</frame_name>

File: src/autonomous_drone/description/quadcopter.urdf.xacro (robot description, xacro)
@@ -319,6 +319,6 @@
 	</link>
 <!-- ======================================================== -->
-    <!-- Define the joint between the base and footprint -->
-	<joint name="base_footprint_joint" type="fixed">
+   <!-- Define joint between base and footprint -->
+   <joint name="base_footprint_joint" type="fixed">
         <parent link="base_link"/>
         <child link="base_footprint"/>
